Commit message: Updated xacro args in both URDF and launch files.

File: teeterbot_description/urdf/teeterbot.urdf.xacro (robot description, xacro)
@@ -20,5 +20,4 @@
   <xacro:property name="body_depth" value="$(arg body_depth)" />
   <xacro:property name="body_length" value="$(arg body_length)" />
-  <xacro:property name="body_com_height" value="${wheel_radius + body_length/2}" />
   <gazebo>
     <plugin name="controller_interface" filename="libteeterbot_controller_interface.so">
@@ -82,5 +81,5 @@
       <origin xyz="0 0 0" rpy="0 0 0"/>
       <geometry>
-        <box size="0.3 0.3 ${body_length}"/>
+        <box size="${body_depth} ${body_width} ${body_length}"/>
       </geometry>
       <material name="orange"/>
@@ -89,5 +88,5 @@
       <origin xyz="0 0 0" rpy="0 0 0"/>
       <geometry>
-        <box size="0.3 0.3 ${body_length}"/>
+        <box size="${body_depth} ${body_width} ${body_length}"/>
       </geometry>
     </collision>
@@ -115,5 +114,5 @@
   </link>
   <joint name="base_com" type="fixed">
-    <origin xyz="0 0 ${body_com_height-wheel_radius}" rpy="0 0 0"/>
+    <origin xyz="0 0 ${body_length/2}" rpy="0 0 0"/>
     <parent link="base_link"/>
     <child link="body_com"/>

Commit message: Changed URDF model to make it work in ROS Noetic / Gazebo 11

File: teeterbot_description/urdf/teeterbot.urdf.xacro (robot description, xacro)
@@ -40,5 +40,5 @@
       <robotNamespace>$(arg robot_name)</robotNamespace>
       <jointName>
-          left_wheel, right_wheel
+          left_wheel_joint, right_wheel_joint
       </jointName>
       <updateRate>100</updateRate>
@@ -74,5 +74,5 @@
       </collision>
     </link>
-    <joint name="${name}" type="continuous">
+    <joint name="${name}_joint" type="continuous">
       <origin xyz="0 ${y_offset} 0" rpy="-1.570796 0 0"/>
       <parent link="base_link"/>
@@ -81,6 +81,6 @@
     </joint>
   </xacro:macro>
-  <wheel name="left_wheel" y_offset="${wheelbase/2}" />
-  <wheel name="right_wheel" y_offset="${-wheelbase/2}" />
+  <xacro:wheel name="left_wheel" y_offset="${wheelbase/2}" />
+  <xacro:wheel name="right_wheel" y_offset="${-wheelbase/2}" />
   <link name="body_com">
     <inertial>
@@ -104,9 +104,4 @@
   </link>
   <link name="base_link">
-    <inertial>
-      <origin xyz="0 0 0" rpy="0 0 0"/>
-      <mass value="0.01"/>
-      <inertia ixx="0.01" ixy="0" ixz="0" iyy="0.01" iyz="0" izz="0.01"/>
-    </inertial>
     <xacro:if value="$(arg training_wheels)" >
       <collision name="training_wheel_1">
@@ -124,5 +119,5 @@
     </xacro:if>
   </link>
-  <joint name="base_com" type="fixed">
+  <joint name="base_com_joint" type="fixed">
     <origin xyz="0 0 ${body_length/2}" rpy="0 0 0"/>
     <parent link="base_link"/>
